File: PDC_new.kicad_sch (KiCad schematic)
At the start: 28 parts, among them J1 Conn_01x02_Pin, J10 Conn_01x02_Pin, J11 XT90PW-F, J12 Conn_01x02_Pin, J2 Conn_01x02_Pin, J3 Conn_01x02_Pin, J4 Conn_01x02_Pin, J5 Conn_01x02_Pin, J6 Conn_01x02_Pin, J7 Conn_01x02_Pin, J8 Conn_01x02_Pin, J9 Conn_01x02_Pin, U1 TPSI3050QDWZRQ1, U10 LM393LVDR, U2 TPSI3050QDWZRQ1, U3 TPSI3050QDWZRQ1, U4 74HC74, U5 URB4805LD-60WR3, U7 NE555D, U8 74HC08, U9 SN74HC14DR

Commit message: Replace SMCJ54CA-13-F TVS diode with SMCJ54A in PDC schematic
Co-Authored-By: Claude Opus 5.5 <noreply@anthropic.com>
Parts:
- removed D1: SMCJ54CA-13-F, SMCJ54CA-13-F:TVS_SMCJ54CA-13-F, symbol SMCJ54CA:SMCJ54CA-13-F
- added D2: SMCJ54A, SMCJ54A:DIOM6859X262N, symbol SMCJ54A:SMCJ54A
Changed lines of the file:
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@@
 	)
 	(symbol
-		(lib_id "SMCJ54CA:SMCJ54CA-13-F")
-		(at 191.77 138.43 0)
+		(lib_id "SMCJ54A:SMCJ54A")
+		(at 170.18 144.78 0)
 		(unit 1)
 		(body_style 1)
@@
 		(dnp no)
 		(fields_autoplaced yes)
-		(property "Reference" "D1"
-			(at 191.77 132.08 0)
-			(show_name no)
-			(do_not_autoplace no)
-			(effects
-				(font
-					(size 1.27 1.27)
-				)
-			)
-		)
-		(property "Value" "SMCJ54CA-13-F"
-			(at 191.77 134.62 0)
-			(show_name no)
-			(do_not_autoplace no)
-			(effects
-				(font
-					(size 1.27 1.27)
-				)
-			)
-		)
-		(property "Footprint" "SMCJ54CA-13-F:TVS_SMCJ54CA-13-F"
-			(at 191.77 138.43 0)
+		(property "Reference" "D2"
+			(at 170.18 138.43 0)
+			(show_name no)
+			(do_not_autoplace no)
+			(effects
+				(font
+					(size 1.27 1.27)
+				)
+			)
+		)
+		(property "Value" "SMCJ54A"
+			(at 170.18 140.97 0)
+			(show_name no)
+			(do_not_autoplace no)
+			(effects
+				(font
+					(size 1.27 1.27)
+				)
+			)
+		)
+		(property "Footprint" "SMCJ54A:DIOM6859X262N"
+			(at 170.18 144.78 0)
 			(hide yes)
 			(show_name no)
@@
 		)
 		(property "Datasheet" ""
-			(at 191.77 138.43 0)
-			(hide yes)
-			(show_name no)
-			(do_not_autoplace no)
-			(effects
-				(font
-					(size 1.27 1.27)
-				)
-			)
-		)
-		(property "Description" "87.1V Clamp 17.2A Ipp Tvs Diode Surface Mount SMC"
-			(at 191.77 138.43 0)
-			(hide yes)
-			(show_name no)
-			(do_not_autoplace no)
-			(effects
-				(font
-					(size 1.27 1.27)
-				)
-				(justify bottom)
-			)
-		)
-		(property "MF" "Diodes Inc."
-			(at 191.77 138.43 0)
-			(hide yes)
-			(show_name no)
-			(do_not_autoplace no)
-			(effects
-				(font
-					(size 1.27 1.27)
-				)
-				(justify bottom)
-			)
-		)
-		(property "MAXIMUM_PACKAGE_HEIGHT" "2.5mm"
-			(at 191.77 138.43 0)
-			(hide yes)
-			(show_name no)
-			(do_not_autoplace no)
-			(effects
-				(font
-					(size 1.27 1.27)
-				)
-				(justify bottom)
-			)
-		)
-		(property "CREATOR" "AMINA"
-			(at 191.77 138.43 0)
+			(at 170.18 144.78 0)
+			(hide yes)
+			(show_name no)
+			(do_not_autoplace no)
+			(effects
+				(font
+					(size 1.27 1.27)
+				)
+			)
+		)
+		(property "Description" "1500W, 54V, Unidirectional, TVS"
+			(at 170.18 144.78 0)
+			(hide yes)
+			(show_name no)
+			(do_not_autoplace no)
+			(effects
+				(font
+					(size 1.27 1.27)
+				)
+				(justify bottom)
+			)
+		)
+		(property "MF" "Taiwan Semiconductor Corporation"
+			(at 170.18 144.78 0)
+			(hide yes)
+			(show_name no)
+			(do_not_autoplace no)
+			(effects
+				(font
+					(size 1.27 1.27)
+				)
+				(justify bottom)
+			)
+		)
+		(property "MAXIMUM_PACKAGE_HEIGHT" "2.62 mm"
+			(at 170.18 144.78 0)
+			(hide yes)
+			(show_name no)
+			(do_not_autoplace no)
+			(effects
+				(font
+					(size 1.27 1.27)
+				)
+				(justify bottom)
+			)
+		)
+		(property "Package" "SMC-2 Taiwan Semiconductor"
+			(at 170.18 144.78 0)
 			(hide yes)
 			(show_name no)
@@
 		)
 		(property "Price" "None"
-			(at 191.77 138.43 0)
-			(hide yes)
-			(show_name no)
-			(do_not_autoplace no)
-			(effects
-				(font
-					(size 1.27 1.27)
-				)
-				(justify bottom)
-			)
-		)
-		(property "Package" "DO-214 Diodes Inc."
-			(at 191.77 138.43 0)
-			(hide yes)
-			(show_name no)
-			(do_not_autoplace no)
-			(effects
-				(font
-					(size 1.27 1.27)
-				)
-				(justify bottom)
-			)
-		)
-		(property "Check_prices" "https://www.snapeda.com/parts/SMCJ54CA-13-F/Diodes+Inc./view-part/?ref=eda"
-			(at 191.77 138.43 0)
-			(hide yes)
-			(show_name no)
-			(do_not_autoplace no)
-			(effects
-				(font
-					(size 1.27 1.27)
-				)
-				(justify bottom)
-			)
-		)
-		(property "DUPLICATE" "SMCJ9.0CA-13-F-,- SMCJ43CA-13-F-,- SMCJ130CA-13-F-,- SMCJ150CA-13-,- SMCJ8.5CA-13-,- SMCJ8.0CA-13-,- SMCJ6.5CA-13-,- SMCJ64CA-13-,- SMCJ26CA-13-F-,- SMCJ36CAQ-13-F-,- SMCJ36CA-13-,- SMCJ30CA-13-F-,- SMCJ120CA-13-F-,- SMCJ6.5CA-13-F-,- SMCJ33CAQ-13-F-,- SMCJ78CA-13-,- SMCJ26CA-13-,- SMCJ15CAQ-13-F-,- SMCJ11CA-13-F-,- SMCJ6.0CA-13-,- SMCJ8.5CA-13-F-,- SMCJ30CA-13-,- SMCJ160CA-13-F-,- SMCJ33CA-13-F-,- SMCJ17CA-13-F-,- SMCJ13CA-13-F-,- SMCJ130CA-13-,- SMCJ120CA-13-,- SMCJ160CA-13-,- SMCJ12CA-13-F-,- SMCJ30CAQ-13-F-,- SMCJ40CA-13-,- SMCJ20CA-13-F-,- SMCJ60CA-13-F-,- SMCJ110CA-13-F-,- SMCJ28CA-13-F-,- SMCJ90CA-13-,- SMCJ170CA-13-,- SMCJ51CA-13-,- SMCJ24CAQ-13-F-,- SMCJ170CA-13-F-,- SMCJ7.0CA-13-,- SMCJ24CA-13-,- SMCJ20CA-13-,- SMCJ85CA-13-,- SMCJ14CA-13-,- SMCJ7.5CA-13-,- SMCJ17CAQ-13-F-,- SMCJ45CA-13-,- SMCJ7.5CA-13-F-,- SMCJ18CAQ-13-F-,- SMCJ22CA-13-F-,- SMCJ24CA-13-F-,- SMCJ54CA-13-F-,- SMCJ7.0CA-13-F-,- SMCJ26CAQ-13-F-,- SMCJ26CAQ-,- SMCJ51CA-13-F-,- SMCJ48CA-13-,- SMCJ8.0CA-13-F-,- SMCJ12CA-13-,- SMCJ40CA-13-F-,- SMCJ10CA-13-F-,- SMCJ16CAQ-13-F-,- SMCJ33CA-13-,- SMCJ43CA-13-,- SMCJ60CA-13-,- SMCJ11CA-13-,- SMCJ22CA-13-,- SMCJ10CA-13-,- SMCJ110CA-13-,- SMCJ14CA-13-F-,- SMCJ28CAQ-13-F-,- SMCJ22CAQ-13-F-,- SMCJ17CA-13-,- SMCJ6.0CA-13-F-,- SMCJ5.0CA-13-F-,- SMCJ16CA-13-F-,- SMCJ75CA-13-F-,- SMCJ75CA-13-,- SMCJ15CA-13-F-,- SMCJ18CA-13-F-,- SMCJ70CA-13-F-,- SMCJ70CA-13-,- SMCJ9.0CA-13-,- SMCJ100CA-13-,- SMCJ18CA-13-,- SMCJ15CA-13-,- SMCJ36CA-13-F-,- SMCJ90CA-13-F-,- SMCJ54CA-13-,- SMCJ58CA-13-F-,- SMCJ85CA-13-F-,- SMCJ13CA-13-,- SMCJ58CA-13-,- SMCJ28CA-13-,- SMCJ150CA-13-F-,- SMCJ78CA-13-F-,- SMCJ48CA-13-F-,- SMCJ14CAQ-13-F-,- SMCJ45CA-13-F-,- SMCJ16CA-13-,- SMCJ100CA-13-F-,- SMCJ64CA-13-F-,-"
-			(at 191.77 138.43 0)
-			(hide yes)
-			(show_name no)
-			(do_not_autoplace no)
-			(effects
-				(font
-					(size 1.27 1.27)
-				)
-				(justify bottom)
-			)
-		)
-		(property "STANDARD" "Manufacturer Recommendations"
-			(at 191.77 138.43 0)
-			(hide yes)
-			(show_name no)
-			(do_not_autoplace no)
-			(effects
-				(font
-					(size 1.27 1.27)
-				)
-				(justify bottom)
-			)
-		)
-		(property "PARTREV" "19 - 2"
-			(at 191.77 138.43 0)
-			(hide yes)
-			(show_name no)
-			(do_not_autoplace no)
-			(effects
-				(font
-					(size 1.27 1.27)
-				)
-				(justify bottom)
-			)
-		)
-		(property "VERIFIER" ""
-			(at 191.77 138.43 0)
-			(hide yes)
-			(show_name no)
-			(do_not_autoplace no)
-			(effects
-				(font
-					(size 1.27 1.27)
-				)
-				(justify bottom)
-			)
-		)
-		(property "SnapEDA_Link" "https://www.snapeda.com/parts/SMCJ54CA-13-F/Diodes+Inc./view-part/?ref=snap"
-			(at 191.77 138.43 0)
-			(hide yes)
-			(show_name no)
-			(do_not_autoplace no)
-			(effects
-				(font
-					(size 1.27 1.27)
-				)
-				(justify bottom)
-			)
-		)
-		(property "MP" "SMCJ54CA-13-F"
-			(at 191.77 138.43 0)
-			(hide yes)
-			(show_name no)
-			(do_not_autoplace no)
-			(effects
-				(font
-					(size 1.27 1.27)
-				)
-				(justify bottom)
-			)
-		)
-		(property "Purchase-URL" "https://www.snapeda.com/api/url_track_click_mouser/?unipart_id=835278&manufacturer=Diodes Inc.&part_name=SMCJ54CA-13-F&search_term=smcj54ca"
-			(at 191.77 138.43 0)
+			(at 170.18 144.78 0)
+			(hide yes)
+			(show_name no)
+			(do_not_autoplace no)
+			(effects
+				(font
+					(size 1.27 1.27)
+				)
+				(justify bottom)
+			)
+		)
+		(property "Check_prices" "https://www.snapeda.com/parts/SMCJ54A/taiwan/view-part/?ref=eda"
+			(at 170.18 144.78 0)
+			(hide yes)
+			(show_name no)
+			(do_not_autoplace no)
+			(effects
+				(font
+					(size 1.27 1.27)
+				)
+				(justify bottom)
+			)
+		)
+		(property "STANDARD" "IPC-7351B"
+			(at 170.18 144.78 0)
+			(hide yes)
+			(show_name no)
+			(do_not_autoplace no)
+			(effects
+				(font
+					(size 1.27 1.27)
+				)
+				(justify bottom)
+			)
+		)
+		(property "PARTREV" "R2102"
+			(at 170.18 144.78 0)
+			(hide yes)
+			(show_name no)
+			(do_not_autoplace no)
+			(effects
+				(font
+					(size 1.27 1.27)
+				)
+				(justify bottom)
+			)
+		)
+		(property "SnapEDA_Link" "https://www.snapeda.com/parts/SMCJ54A/taiwan/view-part/?ref=snap"
+			(at 170.18 144.78 0)
+			(hide yes)
+			(show_name no)
+			(do_not_autoplace no)
+			(effects
+				(font
+					(size 1.27 1.27)
+				)
+				(justify bottom)
+			)
+		)
+		(property "MP" "SMCJ54A"
+			(at 170.18 144.78 0)
+			(hide yes)
+			(show_name no)
+			(do_not_autoplace no)
+			(effects
+				(font
+					(size 1.27 1.27)
+				)
+				(justify bottom)
+			)
+		)
+		(property "Purchase-URL" "https://www.snapeda.com/api/url_track_click_mouser/?unipart_id=4811291&manufacturer=Taiwan Semiconductor Corporation&part_name=SMCJ54A&search_term=smcj54a"
+			(at 170.18 144.78 0)
 			(hide yes)
 			(show_name no)
@@
 		)
 		(property "Availability" "In Stock"
-			(at 191.77 138.43 0)
-			(hide yes)
-			(show_name no)
-			(do_not_autoplace no)
-			(effects
-				(font
-					(size 1.27 1.27)
-				)
-				(justify bottom)
-			)
-		)
-		(property "MANUFACTURER" "Diodes Inc."
-			(at 191.77 138.43 0)
-			(hide yes)
-			(show_name no)
-			(do_not_autoplace no)
-			(effects
-				(font
-					(size 1.27 1.27)
-				)
-				(justify bottom)
-			)
-		)
-		(pin "1"
-		)
-		(pin "2"
+			(at 170.18 144.78 0)
+			(hide yes)
+			(show_name no)
+			(do_not_autoplace no)
+			(effects
+				(font
+					(size 1.27 1.27)
+				)
+				(justify bottom)
+			)
+		)
+		(property "MANUFACTURER" "Taiwan Semiconductor"
+			(at 170.18 144.78 0)
+			(hide yes)
+			(show_name no)
+			(do_not_autoplace no)
+			(effects
+				(font
+					(size 1.27 1.27)
+				)
+				(justify bottom)
+			)
+		)
+		(pin "A"
+		)
+		(pin "C"
 		)
 		(instances
 			(project "PDC_new"
 				(path "/671abb5b-543a-4728-a531-5a7ec9a38d76"
-					(reference "D1")
+					(reference "D2")
 					(unit 1)
 				)

Commit message: Add MOSFET switching stage and passive network to PDC schematic
- Add 4x IPB017N10N5ATMA1 power MOSFETs and 2x BSS123 small-signal FETs
- Add 3 more 3568-15 fuses and a second XT90PW-F connector
- Add resistors (23), capacitors (6 ceramic, 5 more polarized),
  2 diodes and a status LED
- Add GND power symbols and wire up the circuit
- Project: relax ERC pin_not_connected, pin_not_driven and
  power_pin_not_driven from error to ignore

Co-Authored-By: Claude Opus 5.5 <noreply@anthropic.com>
Parts:
- added C10, C11, C12, C13, C14, C15: C, symbol Device:C
- added C5: 1000uF/100V, Capacitor_THT:CP_Radial_D18.0mm_P7.50mm, symbol Device:C_Polarized
- added C6: 100uF/100V, Capacitor_THT:CP_Radial_D18.0mm_P7.50mm, symbol Device:C_Polarized
- added C7, C8, C9: 1uF/100V, Capacitor_THT:CP_Radial_D18.0mm_P7.50mm, symbol Device:C_Polarized
- added D1, D3: D, symbol Device:D
- added D4: LED, symbol Device:LED
- added F2, F3, F4: 3568-15, fuse:FUSE_3568-15, symbol 3568-15:3568-15
- added J13: XT90PW-F, XT90PW-F:AMASS_XT90PW-F, symbol XT90I:XT90PW-F
- added Q1, Q5: BSS123, Package_TO_SOT_SMD:SOT-23, symbol Transistor_FET:BSS123
- added R1, R2: R, symbol Device:R
- added R10, R11, R12, R13, R21, R22, R23, R8: 10k, symbol Device:R
- added R14, R15, R16, R17, R7, R9: 10, symbol Device:R
- added R18, R19, R20: 20k, symbol Device:R
- added R3: 47k, symbol Device:R
- added R4: 158k, symbol Device:R
- added R5: 22k, symbol Device:R
- added R6: 150k, symbol Device:R
- added U11(main), U12(main), U14(main), U6(main): IPB017N10N5ATMA1, IPB017N10N5ATMA1_INF, symbol IPB017N10N5ATMA1:IPB017N10N5ATMA1
- C1, C2, C3, C4: value C_Polarized -> 1000uF/100V; footprint (none) -> Capacitor_THT:CP_Radial_D18.0mm_P7.50mm
- U7: value NE555D -> TLC555CDR
Connections:
- net GND: now reaches J11.N (NEG)
- net GND: now also C1.2, C2.2, C3.2, C4.2, D2.A, J1.2 (Pin_2), J10.2 (Pin_2), J12.2 (Pin_2), J2.2 (Pin_2), J3.2 (Pin_2), J4.2 (Pin_2), J5.2 (Pin_2), J6.2 (Pin_2), J7.2 (Pin_2), J8.2 (Pin_2), J9.2 (Pin_2), U1.4 (VSSP), U10.4 (GND), U2.4 (VSSP), U3.4 (VSSP), U3.5 (VSSS), U5.2 (GND), C15.2, C5.2, C6.2, C7.1, C8.1, C9.1, D4.1 (K), J13.N (NEG), Q1.2 (S), R18.2, R19.2, R20.2, R21.1, R22.2, R3.1, R8.2
- net at J11.P (POS): now also D2.C, F1.2, F1.4, C5.1, D1.2 (A), F3.1, F3.3, R3.2, R4.2, U11(main).4, U12(main).4, U14(main).4, U6(main).4
- net at U3.2 (PXFR): now also R19.1
- net at U3.3 (VDDP): now also C8.2
- net at U3.6 (VDDM): now also C14.2, C15.1
- net at U3.7 (VDDH): now also C14.1
- net at U3.8 (VDRV): now also R7.2
- net at J6.1 (Pin_1): now also C1.1, C2.1, C3.1, C4.1, J1.1 (Pin_1), J10.1 (Pin_1), J2.1 (Pin_1), J3.1 (Pin_1), J4.1 (Pin_1), J5.1 (Pin_1), J7.1 (Pin_1), J8.1 (Pin_1), J9.1 (Pin_1), U1.5 (VSSS), U2.5 (VSSS), C11.2, C13.2, D3.2 (A), Q5.2 (S), R11.1, R12.1, R13.1, R2.2, R23.1, R5.1, R6.1, U11(main).2, U11(main).3, U11(main).5, U11(main).6, U11(main).7, U12(main).2, U12(main).3, U12(main).5, U12(main).6, U12(main).7, U14(main).2, U14(main).3, U14(main).5, U14(main).6, U14(main).7, U6(main).2, U6(main).3, U6(main).5, U6(main).6, U6(main).7
- net at J12.1 (Pin_1): now also F4.1, F4.3
- net at U5.3 (Vin): now also C6.1, F2.2, F2.4
- net at U5.4 (+Vo): now also F4.2, F4.4
- net at U2.2 (PXFR): now also R20.1
- net at U2.3 (VDDP): now also C9.2
- net at U2.6 (VDDM): now also C12.2, C13.1
- net at U2.7 (VDDH): now also C12.1
- net at U2.8 (VDRV): now also R14.2, R15.2, R16.2, R17.2
- net at U10.2 (IN1-): now also R22.1, R6.2
- net at U10.3 (IN1+): now also R21.2, R4.1
- net at U1.2 (PXFR): now also R18.1
- net at U1.3 (VDDP): now also C7.2
- net at U1.6 (VDDM): now also C10.2, C11.1
- net at U1.7 (VDDH): now also C10.1
- net at U1.8 (VDRV): now also R9.2
- net at F1.1, F1.3: now also J13.P (POS)
- new net: R12.2, R15.1, U12(main).1
- new net: R13.2, R14.1, U6(main).1
- new net: Q1.1 (G), R7.1, R8.1
- new net: D4.2 (A), R5.2
- new net: Q5.1 (G), R10.1, R9.1
- new net: Q5.3 (D), R1.2, R10.2
- new net: F3.2, F3.4, R1.1
- new net: R17.1, R23.2, U11(main).1
- new net: Q1.3 (D), R2.1
- new net: R11.2, R16.1, U14(main).1
- new net: D1.1 (K), D3.1 (K), F2.1, F2.3
Other:
- note added: "Bat+"
- note added: "Batt In"
- note added: "Bus+"
- note added: "Precharge circuit"
- moved on the sheet: C1, D2, F1, J1, J10, J11, J12, J2, J3, J4, J5, J6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
