File: PDC_new.kicad_sch (KiCad schematic)
At the start: 17 parts, among them J1 Conn_01x02, J10 Conn_01x02, J2 Conn_01x02, J3 Conn_01x02, J4 Conn_01x02, J5 Conn_01x02, J6 Conn_01x02, J7 Conn_01x02, J8 Conn_01x02, J9 Conn_01x02

Commit message: Update PDC schematic: add SMCJ54A TVS and SN74HC08D AND gate, A3 sheet
Ignore locally imported SMCJ54A/SN74HC08D symbol and footprint libraries.
Parts:
- removed Bat, J1, J10, J2, J3, J4, J5, J6, J7, J8, J9, To_pi/stm32: Conn_01x02, symbol Connector_Generic:Conn_01x02
- removed U1: (no value), TPSI3050-Q1:SOIC-8_DWZ_7.5x5.85mm_P1.27mm, symbol TPSI3050-Q1:_1
- added C10, C11, C12, C13, C14, C15, C16: C, symbol Device:C
- added C17: 10nF, symbol Device:C
- added C18: 100nF, symbol Device:C
- added C19: 0.47 µF, symbol Device:C
- added C20: 2.2 µF, symbol Device:C
- added C21: 47nF, symbol Device:C
- added C5: 1000uF/100V, Capacitor_THT:CP_Radial_D18.0mm_P7.50mm, symbol Device:C_Polarized
- added C6: 100uF/100V, Capacitor_THT:CP_Radial_D18.0mm_P7.50mm, symbol Device:C_Polarized
- added C7, C8, C9: 1uF/100V, Capacitor_THT:CP_Radial_D18.0mm_P7.50mm, symbol Device:C_Polarized
- added D1, D3: D, symbol Device:D
- added D2: SMCJ54A, SMCJ54A:DIOM6859X262N, symbol SMCJ54A:SMCJ54A
- added D4: LED, symbol Device:LED
- added D5: 1N4148W, Diode_SMD:D_SOD-123, symbol Diode:1N4148W
- added F1, F2, F3, F4: 3568-15, fuse:FUSE_3568-15, symbol 3568-15:3568-15
- added J1, J10, J2, J3, J4, J5, J6, J7, J8, J9: Conn_01x02_Pin, Connector_AMASS:AMASS_XT60PW-F_1x02_P7.20mm_Horizontal, symbol Connector:Conn_01x02_Pin
- added J11, J13: XT90PW-F, XT90PW-F:AMASS_XT90PW-F, symbol XT90I:XT90PW-F
- added J12: Conn_01x02_Pin, Connector_AMASS:AMASS_XT30PW-F_1x02_P2.50mm_Horizontal, symbol Connector:Conn_01x02_Pin
- added Q1, Q5: BSS123, Package_TO_SOT_SMD:SOT-23, symbol Transistor_FET:BSS123
- added R1, R2: R, symbol Device:R
- added R10, R11, R12, R13, R21, R22, R23, R25, R26, R8: 10k, symbol Device:R
- added R14, R15, R16, R17, R7, R9: 10, symbol Device:R
- added R18, R19, R20: 20k, symbol Device:R
- added R24: 1M, symbol Device:R
- added R27: 100k, symbol Device:R
- added R3: 47k, symbol Device:R
- added R4: 158k, symbol Device:R
- added R5: 22k, symbol Device:R
- added R6: 150k, symbol Device:R
- added RV1: 500k, Potentiometer_THT:Potentiometer_Bourns_3296W_Vertical, symbol Device:R_Potentiometer_Trim
- added U1, U2, U3: TPSI3050QDWZRQ1, TPSI3050_Q1:DWZ0008A-MFG, symbol TPSI3050_Q1:TPSI3050QDWZRQ1
- added U10: LM393LVDR, D0008A-IPC_A, symbol LM393LVDR:LM393LVDR
- added U11(main), U12(main), U14(main), U6(main): IPB017N10N5ATMA1, IPB017N10N5ATMA1_INF, symbol IPB017N10N5ATMA1:IPB017N10N5ATMA1
- added U4: 74HC74, symbol 74xx:74HC74
- added U5: URB4805LD-60WR3, NexusPDB:URB4805LD-60WR3, symbol URB48_LD-60WR3:URB4805LD-60WR3
- added U7: TLC555CDR, Package_SO:SOIC-8_3.9x4.9mm_P1.27mm, symbol Timer:NE555D
- added U8: SN74HC08D, SN74HC08D:SOIC127P600X175-14N, symbol SN74HC08D:SN74HC08D
- added U9: SN74HC14DR, SN74HC14DR:SOIC127P600X175-14N, symbol SN74HC14DR:SN74HC14DR
- C1, C2, C3, C4: value C_Polarized -> 1000uF/100V; footprint (none) -> Capacitor_THT:CP_Radial_D18.0mm_P7.50mm
Connections:
- net at C1.1: now also C2.1, C3.1, C4.1, C11.2, C13.2, D3.2 (A), J1.1 (Pin_1), J10.1 (Pin_1), J2.1 (Pin_1), J3.1 (Pin_1), J4.1 (Pin_1), J5.1 (Pin_1), J6.1 (Pin_1), J7.1 (Pin_1), J8.1 (Pin_1), J9.1 (Pin_1), Q5.2 (S), R11.1, R12.1, R13.1, R2.2, R23.1, R5.1, R6.1, U1.5 (VSSS), U11(main).2, U11(main).3, U11(main).5, U11(main).6, U11(main).7, U12(main).2, U12(main).3, U12(main).5, U12(main).6, U12(main).7, U14(main).2, U14(main).3, U14(main).5, U14(main).6, U14(main).7, U2.5 (VSSS), U6(main).2, U6(main).3, U6(main).5, U6(main).6, U6(main).7
- net GND: now reaches C1.2
- net GND: now also C2.2, C3.2, C4.2, C15.2, C16.2, C17.1, C19.1, C20.1, C5.2, C6.2, C7.1, C8.1, C9.1, D2.A, D4.1 (K), J1.2 (Pin_2), J10.2 (Pin_2), J11.N (NEG), J12.2 (Pin_2), J13.N (NEG), J2.2 (Pin_2), J3.2 (Pin_2), J4.2 (Pin_2), J5.2 (Pin_2), J6.2 (Pin_2), J7.2 (Pin_2), J8.2 (Pin_2), J9.2 (Pin_2), Q1.2 (S), R18.2, R19.2, R20.2, R21.1, R22.2, R27.2, R3.1, R8.2, U1.4 (VSSP), U10.4 (GND), U2.4 (VSSP), U3.4 (VSSP), U3.5 (VSSS), U4.7 (GND), U5.2 (GND), U7.1 (GND), U9.7 (GND)
- new net: R12.2, R15.1, U12(main).1
- new net: C5.1, D1.2 (A), D2.C, F1.2, F1.4, F3.1, F3.3, J11.P (POS), R3.2, R4.2, U11(main).4, U12(main).4, U14(main).4, U6(main).4
- new net: C8.2, U3.1 (EN), U3.3 (VDDP), U9.10 (5Y)
- new net: R19.1, U3.2 (PXFR)
- new net: C14.2, C15.1, U3.6 (VDDM)
- new net: C14.1, U3.7 (VDDH)
- new net: R7.2, U3.8 (VDRV)
- new net: C10.2, C11.1, U1.6 (VDDM)
- new net: C20.2, R25.1, R26.2, U10.1 (OUT1)
- new net: R25.2, U9.1 (1A)
- new net: R13.2, R14.1, U6(main).1
- new net: Q1.1 (G), R7.1, R8.1
- new net: D5.1 (K), R24.2, U8.1 (1A), U9.6 (3Y)
- new net: U8.10 (3B), U9.4 (2Y)
- new net: U4.6 (~{Q}), U8.13 (4B)
- new net: U8.3 (1Y), U9.11 (5A)
- new net: U4.13 (~{R}), U8.5 (2B), U9.12 (6Y)
- new net: U4.1 (~{R}), U8.6 (2Y)
- new net: U4.11 (C), U8.8 (3Y)
- new net: U8.9 (3A), U9.8 (4Y)
- new net: D4.2 (A), R5.2
- new net: C18.1, C21.2, F4.2, F4.4, R26.1, U4.10 (~{S}), U4.12 (D), U4.14 (VCC), U4.4 (~{S}), U5.4 (+Vo), U7.4 (~{RST})
- new net: Q5.1 (G), R10.1, R9.1
- new net: Q5.3 (D), R1.2, R10.2
- new net: F3.2, F3.4, R1.1
- new net: R18.1, U1.2 (PXFR)
- new net: F4.1, F4.3, J12.1 (Pin_1)
- new net: C21.1, R27.1, U9.13 (6A)
- new net: C16.1, U9.14 (VCC)
- new net: U4.2 (D), U4.3 (C), U4.8 (~{Q}), U9.2 (1Y), U9.3 (2A)
- new net: U7.3 (OUT), U9.9 (4A)
- new net: R17.1, R23.2, U11(main).1
- new net: R14.2, R15.2, R16.2, R17.2, U2.8 (VDRV)
- new net: Q1.3 (D), R2.1
- new net: C7.2, U1.3 (VDDP)
- new net: C18.2, U7.8 (VCC)
- new net: C19.2, D5.2 (A), R24.1, U7.2 (TRIG), U7.6 (THRES)
- new net: R11.2, R16.1, U14(main).1
- new net: C6.1, F2.2, F2.4, U5.3 (Vin)
- new net: RV1.2, RV1.3, U5.5 (0V)
- new net: RV1.1, U5.6 (Trim)
- new net: U2.1 (EN), U4.5 (Q)
- new net: D1.1 (K), D3.1 (K), F2.1, F2.3
- new net: C17.2, U7.5 (CONT)
- new net: R22.1, R6.2, U10.2 (IN1-)
- new net: R21.2, R4.1, U10.3 (IN1+)
- new net: C12.2, C13.1, U2.6 (VDDM)
- new net: R20.1, U2.2 (PXFR)
- new net: C9.2, U2.3 (VDDP)
- new net: C12.1, U2.7 (VDDH)
- new net: F1.1, F1.3, J13.P (POS)
- new net: C10.1, U1.7 (VDDH)
- new net: R9.2, U1.8 (VDRV)
- no-connect marks 0 -> 2
Other:
- note added: "Bat+"
- note added: "Batt In"
- note added: "Bus+"
- note added: "Precharge circuit"
- moved on the sheet: C1
