File: PDC_new.kicad_sch (KiCad schematic)
At the start: 86 parts, among them J1 Conn_01x02_Pin, J10 Conn_01x02_Pin, J11 XT90PW-F, J12 Conn_01x02_Pin, J13 XT90PW-F, J2 Conn_01x02_Pin, J3 Conn_01x02_Pin, J4 Conn_01x02_Pin, J5 Conn_01x02_Pin, J6 Conn_01x02_Pin, J7 Conn_01x02_Pin, J8 Conn_01x02_Pin, J9 Conn_01x02_Pin, Q1 BSS123, Q5 BSS123, U1 TPSI3050QDWZRQ1, U10 LM393LVDR, U11(main) IPB017N10N5ATMA1, U12(main) IPB017N10N5ATMA1, U14(main) IPB017N10N5ATMA1, U2 TPSI3050QDWZRQ1, U3 TPSI3050QDWZRQ1, U4 74HC74, U5 URB4805LD-60WR3, U6(main) IPB017N10N5ATMA1, U7 TLC555CDR, U8 SN74HC08D, U9 SN74HC14DR

Commit message: Update PDC schematic: add IRF540N MOSFET, JST XH connector and tactile switch
- Add IRF540NSTRLPBF N-channel MOSFET, B2B-XH-A JST XH 2-pin connector
  and TS-1187A tactile switch to the PDC schematic
- Add symbol libraries, footprints and 3D models for the new parts

Co-Authored-By: Claude Opus 5.5 <noreply@anthropic.com>
Parts:
- removed C7, C8: 1uF/100V, Capacitor_THT:CP_Radial_D18.0mm_P7.50mm, symbol Device:C_Polarized
- removed D4: LED, symbol Device:LED
- removed Q5: BSS123, Package_TO_SOT_SMD:SOT-23, symbol Transistor_FET:BSS123
- removed R5: 22k, symbol Device:R
- added C22, C23, C25, C26: 100nF, symbol Device:C
- added C24: 2.2µF, symbol Device:C
- added C8: 1µF, symbol Device:C
- added D6: LED, symbol Device:LED
- added J14: B2B-XH-A__LF__SN_, B2B-XH-A__LF__SN_:JST_B2B-XH-A__LF__SN_, symbol B2B-XH-A__LF__SN_:B2B-XH-A__LF__SN_
- added Q2: IRF540NSTRLPBF, IRF540NSTRLPBF:TRANS_IRF540NSTRLPBF, symbol IRF540NSTRLPBF:IRF540NSTRLPBF
- added R28, R29: 10k, symbol Device:R
- added R30: 22k, symbol Device:R
- added S1: TS-1187A-B-A-B, TS-1187A-B-A-B:SW_TS-1187A-B-A-B, symbol TS-1187A-B-A-B:TS-1187A-B-A-B
- C14, C15: value C -> 470nF
- R1: value R -> 2.7
- R2: value R -> 1k
- renumbered U1 to U1(precharge), U3 to U3(discharge), U5 to U5(buck)
Connections:
- net GND: now also C18.1, U10.5 (IN2+), U8.7 (GND), C22.2, C23.1, C24.2, C25.1, C26.1, C8.1, J14.2
- net at C1.1, C11.2, C13.2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: now also R10.2, Q2.3, R30.1
- net at U3(discharge).1 (EN), U9.10 (5Y): no longer U3(discharge).3 (VDDP)
- net at U8.11 (4Y): now also U1(precharge).1 (EN)
- net at U8.12 (4A): now also U8.3 (1Y), U8.4 (2A), U9.11 (5A)
- net at U8.14 (VCC): now also C16.1, C18.2, C21.2, C9.2, F4.2, F4.4, R26.1, U1(precharge).3 (VDDP), U10.6 (IN2-), U10.8 (VCC), U2.3 (VDDP), U3(discharge).3 (VDDP), U4.10 (~{S}), U4.12 (D), U4.14 (VCC), U4.4 (~{S}), U5(buck).4 (+Vo), U7.4 (~{RST}), U7.8 (VCC), U9.14 (VCC), C22.1, C23.2, C25.2, C26.2, C8.2, R29.2
- net at U8.2 (1B): now also U4.2 (D), U4.8 (~{Q})
- net at R10.1, R9.1: now also Q2.1
- net at R1.2: now also Q2.2; no longer R10.2
- net at C21.1, R27.1, U9.13 (6A): now also S1.A, S1.B
- net at U4.3 (C), U9.2 (1Y), U9.3 (2A): no longer U4.2 (D), U4.8 (~{Q})
- net at U9.5 (3A): now also C24.1, R28.2
- net at Q1.3 (D), R2.1: now also D6.1 (K)
- new net: J14.1, R28.1, R29.1, S1.C, S1.D
- new net: D6.2 (A), R30.2
- no-connect marks 2 -> 5
Other:
- moved on the sheet: C18, C20, C21, C5, D2, Q1, R2, R21, R25, R26, R27, R3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

Commit message: Add footprints, change charging connector and make new connections
- Added footprints and symbols to the PDC schematic, including the new
  XT90 pigtail library (symbol, footprint and preview)
- Changed the charging connector
- Made new connections in the PDC schematic

Co-Authored-By: Claude Opus 5.5 <noreply@anthropic.com>
Parts:
- removed C5: 1000uF/100V, Capacitor_THT:CP_Radial_D18.0mm_P7.50mm, symbol Device:C_Polarized
- removed C6: 100uF/100V, Capacitor_THT:CP_Radial_D18.0mm_P7.50mm, symbol Device:C_Polarized
- removed C9: 1uF/100V, Capacitor_THT:CP_Radial_D18.0mm_P7.50mm, symbol Device:C_Polarized
- removed J11: XT90PW-F, XT90PW-F:AMASS_XT90PW-F, symbol XT90I:XT90PW-F
- added C5: C, Capacitor_THT:CP_Radial_D18.0mm_P7.50mm, symbol Device:C
- added C6: C, Capacitor_THT:CP_Radial_D10.0mm_P5.00mm, symbol Device:C
- added C9: 1µF, Capacitor_SMD:C_0805_2012Metric, symbol Device:C
- added D7: SMF15A, Diode_SMD:D_SMF, symbol Diode:SMF15A
- added J15: Conn_01x02, Connector_JST:JST_XH_B2B-XH-A_1x02_P2.50mm_Vertical, symbol Connector_Generic:Conn_01x02
- added R31: 100, Resistor_SMD:R_0805_2012Metric, symbol Device:R
- added unit 1 of U10
- C10, C11: value C -> 470nF; footprint (none) -> Capacitor_SMD:C_0805_2012Metric
- C12: value C -> 2.2µF; footprint (none) -> Capacitor_SMD:C_0805_2012Metric
- C13: value C -> 2.2 µF; footprint (none) -> Capacitor_SMD:C_1206_3216Metric
- C14: footprint (none) -> Capacitor_SMD:C_1206_3216Metric
- C15, C17, C18, C19, C20, C21, C22, C23, C24, C25, C26, C8: footprint (none) -> Capacitor_SMD:C_0805_2012Metric
- C16: value C -> 1µF; footprint (none) -> Capacitor_SMD:C_0805_2012Metric
- D1, D3: value D -> SS310; footprint (none) -> Diode_SMD:D_SMA
- D6: footprint (none) -> LED_SMD:LED_0805_2012Metric
- R1, R2: footprint (none) -> Resistor_THT:R_Axial_Power_L25.0mm_W9.0mm_P30.48mm
- R10, R11, R12, R13, R14, R15, R16, R17, R18, R19, R20, R21, R22, R23, R24, R25, R26, R27, R28, R29, R3, R4, R6, R7, R8, R9: footprint (none) -> Resistor_SMD:R_0805_2012Metric
- R30: footprint (none) -> Resistor_SMD:R_1206_3216Metric
- renumbered U1(precharge) to U1, U11(main) to U11, U12(main) to U12, U14(main) to U14, U3(discharge) to U3, U5(buck) to U5, U6(main) to U6
Connections:
- net GND: now also C5.1, C6.2, C9.2, D7.2 (A2), J15.2 (Pin_2), U10.4 (GND); no longer U10.4 (GND)
- net at C16.1, C18.2, C21.2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: now also C9.1, U10.8 (VCC); no longer U10.8 (VCC)
- net at D1.2 (A), D2.C, F1.2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: now also C5.2
- net at C20.2, R25.1, R26.2: now also U10.1 (OUT1); no longer U10.1 (OUT1)
- net at U5.1 (Ctrl): now also D7.1 (A1), R31.1
- net at F2.2, F2.4, U5.3 (Vin): now also C6.1
- net at R22.1, R6.2: now also U10.2 (IN1-); no longer U10.2 (IN1-)
- net at R21.2, R4.1: now also U10.3 (IN1+); no longer U10.3 (IN1+)
- new net: J15.1 (Pin_1), R31.2
- no-connect marks 5 -> 4
Other:
- note added: "short pin1,2"
- moved on the sheet: D2, R3

Commit message: Add PDC_new (2) project, URB48 DC-DC libraries and project sym-lib-table
- Add "PDC_new (2)" KiCad project (schematic, PCB, project file)
- Add URB4805LD-60WR3 footprint and URB48_LD-40WR3 Altium source libraries
- Add IRF540NSTRLPBF footprint
- Add project sym-lib-table for local symbol libraries
- Update PDC_new schematic, project settings and fp-lib-table

Co-Authored-By: Claude Opus 5.5 <noreply@anthropic.com>
Parts:
- F1, F2, F3, F4: footprint fuse:FUSE_3568-15 -> Fuse:Fuseholder_Blade_Mini_Keystone_3568
- J14: footprint B2B-XH-A__LF__SN_:JST_B2B-XH-A__LF__SN_ -> Connector_JST:JST_XH_B2B-XH-A_1x02_P2.50mm_Vertical
- U1, U2, U3: footprint TPSI3050_Q1:DWZ0008A-MFG -> ul_TPSI3050QDWZRQ1:DWZ0008A-MFG
- U10: footprint D0008A-IPC_A -> Package_SO:SOIC-8_3.9x4.9mm_P1.27mm
- U11, U12, U14, U6: footprint IPB017N10N5ATMA1_INF -> ul_IPB017N10N5ATMA1:IPB017N10N5ATMA1_INF
- U4: footprint (none) -> Package_SO:SOIC-14_3.9x8.7mm_P1.27mm
- U5: footprint NexusPDB:URB4805LD-60WR3 -> URB4805LD-60WR3:URB48_LD-60WR3
- U9: footprint SN74HC14DR:SOIC127P600X175-14N -> Package_SO:SOIC-14_3.9x8.7mm_P1.27mm
Connections:
- no-connect marks 4 -> 3

Commit message: Link latest schematic and PCB to top-level PDC_new project
Copy the latest PDC_new (2) schematic and routed PCB to PDC_new.kicad_sch
and PDC_new.kicad_pcb, renaming the project/sheetfile references so the
schematic and PCB editors stay in sync under PDC_new.kicad_pro.

Co-Authored-By: Claude Opus 5.5 <noreply@anthropic.com>
Parts:
- removed J15: Conn_01x02, Connector_JST:JST_XH_B2B-XH-A_1x02_P2.50mm_Vertical, symbol Connector_Generic:Conn_01x02
- added U13: XT90PW(2+2)-M.G.Y, XT90I(2+2)PW-M:CONN-TH_XT90PW2X2-MGY, symbol XT90I(2+2)PW-M:XT90PW(2+2)-M.G.Y
Connections:
- net GND: now also U13.1, U13.6
- net BUCK_CTRL: now reaches D7.1 (A1), R31.1, U5.1 (Ctrl)
- net BUS+: now reaches C1.1, C11.2, C13.2, C2.1, C3.1, C4.1, D3.2 (A), J1.1 (Pin_1), J10.1 (Pin_1), J2.1 (Pin_1), J3.1 (Pin_1), J4.1 (Pin_1), J5.1 (Pin_1), J6.1 (Pin_1), J7.1 (Pin_1), J8.1 (Pin_1), J9.1 (Pin_1), Q2.3, R10.2, R11.1, R12.1, R13.1, R2.2, R23.1, R30.1, R6.1, U1.5 (VSSS), U11.2, U11.3, U11.5, U11.6, U12.2, U12.3, U12.5, U12.6, U14.2, U14.3, U14.5, U14.6, U2.5 (VSSS), U6.2, U6.3, U6.5, U6.6
- net BUS+: now also U11.4, U12.4, U14.4, U6.4; no longer U11.7, U12.7, U14.7, U6.7
- net GATE_U12: now reaches R12.2, R15.1, U12.1
- net +5V: now reaches C16.1, C18.2, C21.2, C22.1, C23.2, C25.2, C26.2, C8.2, C9.1, F4.2, F4.4, R26.1, R29.2, U1.3 (VDDP), U10.6 (IN2-), U10.8 (VCC), U2.3 (VDDP), U3.3 (VDDP), U4.10 (~{S}), U4.12 (D), U4.14 (VCC), U4.4 (~{S}), U5.4 (+Vo), U7.4 (~{RST}), U7.8 (VCC), U8.14 (VCC), U9.14 (VCC)
- net MSTR_SW: now reaches J14.1, R28.1, R29.1, S1.C, S1.D
- net MSTR_FILT: now reaches C24.1, R28.2, U9.5 (3A)
- net EN_BLEED: now reaches U3.1 (EN), U9.10 (5Y)
- net at C20.2, R26.2, U10.1 (OUT1): now also R25.2; no longer R25.1
- net CMP_FILT: now reaches U9.1 (1A)
- net CMP_FILT: now also R25.1; no longer R25.2
- net GATE_U6: now reaches R13.2, R14.1, U6.1
- net BATT+: now reaches C5.2, D1.2 (A), D2.C, F1.2, F1.4, F3.1, F3.3, R3.2, R4.2
- net BATT+: now also U11.7, U12.7, U14.7, U6.7, U13.2; no longer U11.4, U12.4, U14.4, U6.4
- net MSTR_ON: now reaches D5.1 (K), R24.2, U8.1 (1A), U9.6 (3Y)
- net DONE_N: now reaches U8.10 (3B), U9.4 (2Y)
- net EN_PRE: now reaches U1.1 (EN), U8.11 (4Y)
- net RUN_OK: now reaches U8.12 (4A), U8.3 (1Y), U8.4 (2A), U9.11 (5A)
- net RUN_N: now reaches U4.6 (~{Q}), U8.13 (4B)
- net FAULT_N: now reaches U4.2 (D), U4.8 (~{Q}), U8.2 (1B)
- net POR_N: now reaches U4.13 (~{R}), U8.5 (2B), U9.12 (6Y)
- net RUN_CLR_N: now reaches U4.1 (~{R}), U8.6 (2Y)
- net FAULT_SET: now reaches U4.11 (C), U8.8 (3Y)
- net TIMEOUT: now reaches U8.9 (3A), U9.8 (4Y)
- net DET: now reaches R31.2
- net DET: now also U13.5
- net POR_RC: now reaches C21.1, R27.1, S1.A, S1.B, U9.13 (6A)
- net PC_DONE: now reaches U4.3 (C), U9.2 (1Y), U9.3 (2A)
- net TMR_OUT: now reaches U7.3 (OUT), U9.9 (4A)
- net GATE_U11: now reaches R17.1, R23.2, U11.1
- net GATE_MAIN: now reaches R14.2, R15.2, R16.2, R17.2, U2.8 (VDRV)
- net TIMER_RC: now reaches C19.2, D5.2 (A), R24.1, U7.2 (TRIG), U7.6 (THRES)
- net GATE_U14: now reaches R11.2, R16.1, U14.1
- net EN_MAIN: now reaches U2.1 (EN), U4.5 (Q)
- net BUS_SENSE: now reaches R22.1, R6.2, U10.2 (IN1-)
- net BATT_SENSE: now reaches R21.2, R4.1, U10.3 (IN1+)
- no-connect marks 3 -> 5
Other:
- note added: "Buck to 5V"
- note added: "Decoupling caps + sensing"
- note added: "bus capacitors"
- note added: "charging circut"
- note added: "comparator logic"
- note added: "discharge circuit"
- note added: "mainbus circut"
- note added: "masterswitch circut"
- note added: "output to all the actuators"
- note removed: "Bat+"
- note removed: "Bus+"
- note removed: "short pin1,2"
- moved on the sheet: C1, C10, C11, C12, C13, C14, C15, C16, C17, C18, C19, C2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

Commit message: Reorganize repo: move libraries into Libraries/, promote PDC_new (2) to main project
Libraries:
- Move all symbol/footprint folders into Libraries/: B2B-XH-A__LF__SN_,
  IRF540NSTRLPBF, SMCJ54A, SMCJ54CA-13-F, SN74HC08D, SN74HC14DR,
  TS-1187A-B-A-B, XT90PW-F, ul_LM393LVDR and pdc_new.pretty.
- Merge root ul_IPB017N10N5ATMA1/ and ul_TPSI3050QDWZRQ1/ into the existing
  folders in Libraries/ (KiCADv6 symbols/footprints moved in; duplicate
  readme.txt and ImportGuides.html at the root dropped).
- Update fp-lib-table and sym-lib-table to point at ${KIPRJMOD}/Libraries/.

Project files:
- Replace PDC_new.kicad_sch/.kicad_pcb/.kicad_pro with the latest
  PDC_new (2) versions and remove the PDC_new (2)/ folder.
- Move PDC_new (2)/report.txt to the repo root.
- Remove the stray extensionless "PDC_new" file (old schematic copy).
- Rename internal "PDC_new (2)" references (schematic instance project
  names, PCB sheetfile refs, project metadata) to "PDC_new".
- Change absolute C:/Users/... 3D model paths in the PCB to
  ${KIPRJMOD}/Libraries/... so they resolve on any machine.

Other:
- .history/ is already ignored by .gitignore (applies at any depth).
- Update README to describe the Libraries/ folder.

Co-Authored-By: Claude Opus 5.5 <noreply@anthropic.com>
Parts:
- removed C14: 470nF, Capacitor_SMD:C_1206_3216Metric, symbol Device:C
- removed C15: 470nF, Capacitor_SMD:C_0805_2012Metric, symbol Device:C
- removed C24: 2.2µF, Capacitor_SMD:C_0805_2012Metric, symbol Device:C
- removed C8: 1µF, Capacitor_SMD:C_0805_2012Metric, symbol Device:C
- removed D6: LED, LED_SMD:LED_0805_2012Metric, symbol Device:LED
- removed F2, F3: 3568-15, Fuse:Fuseholder_Blade_Mini_Keystone_3568, symbol 3568-15:3568-15
- removed J14: B2B-XH-A__LF__SN_, Connector_JST:JST_XH_B2B-XH-A_1x02_P2.50mm_Vertical, symbol B2B-XH-A__LF__SN_:B2B-XH-A__LF__SN_
- removed Q1: BSS123, Package_TO_SOT_SMD:SOT-23, symbol Transistor_FET:BSS123
- removed R19: 20k, Resistor_SMD:R_0805_2012Metric, symbol Device:R
- removed R2: 1k, Resistor_THT:R_Axial_Power_L25.0mm_W9.0mm_P30.48mm, symbol Device:R
- removed R28, R29, R8: 10k, Resistor_SMD:R_0805_2012Metric, symbol Device:R
- removed R30: 22k, Resistor_SMD:R_1206_3216Metric, symbol Device:R
- removed S1: TS-1187A-B-A-B, TS-1187A-B-A-B:SW_TS-1187A-B-A-B, symbol TS-1187A-B-A-B:TS-1187A-B-A-B
- removed U3: TPSI3050QDWZRQ1, ul_TPSI3050QDWZRQ1:DWZ0008A-MFG, symbol TPSI3050_Q1:TPSI3050QDWZRQ1
- added D4: LED, LED_SMD:LED_0805_2012Metric, symbol Device:LED
- added J14, J15: Conn_01x02_Pin, Connector_AMASS:AMASS_XT60PW-F_1x02_P7.20mm_Horizontal, symbol Connector:Conn_01x02_Pin
- added R5: 10k, Resistor_THT:R_Axial_Power_L25.0mm_W9.0mm_P30.48mm, symbol Device:R
- C10, C11, C9: footprint Capacitor_SMD:C_0805_2012Metric -> LED_SMD:LED_0805_2012Metric_Pad1.15x1.40mm_HandSolder
- C12: value 2.2µF -> 4.3µF; footprint Capacitor_SMD:C_0805_2012Metric -> Capacitor_SMD:C_1206_3216Metric_Pad1.33x1.80mm_HandSolder
- C13: value 2.2 µF -> 4.3 µF; footprint Capacitor_SMD:C_1206_3216Metric -> Capacitor_SMD:C_1206_3216Metric_Pad1.33x1.80mm_HandSolder
- C16, C17, C18, C19, C20, C21, C22, C23, C25, C26: footprint Capacitor_SMD:C_0805_2012Metric -> Capacitor_SMD:C_0805_2012Metric_Pad1.18x1.45mm_HandSolder
- C5, C6: value C -> 100uF
- J11: renamed from U13; footprint XT90I(2+2)PW-M:CONN-TH_XT90PW2X2-MGY -> XT90PW(2+2)-M.G.Y:CONN-TH_XT90PW2X2-MGY
- J13: value XT90PW-F -> QS8; footprint XT90PW-F:AMASS_XT90PW-F -> QS8_S_Connectors:QS8-S-M_Vertical_DirectCup
- R10, R11, R12, R13, R14, R15, R16, R17, R18, R20, R21, R22, R23, R24, R25, R26, R27, R31, R4, R6, R9: footprint Resistor_SMD:R_0805_2012Metric -> Resistor_SMD:R_0805_2012Metric_Pad1.20x1.40mm_HandSolder
- R3: footprint Resistor_SMD:R_0805_2012Metric -> Resistor_SMD:R_1206_3216Metric_Pad1.30x1.75mm_HandSolder
- R7: value 10 -> 22k; footprint Resistor_SMD:R_0805_2012Metric -> Resistor_SMD:R_1206_3216Metric_Pad1.30x1.75mm_HandSolder
Connections:
- net MSTR_FILT is gone; now on net GND: U9.5 (3A)
- net BATT+: now also R1.1
- net BUS+: now also D4.2 (A), J14.1 (Pin_1), J15.1 (Pin_1), R5.2
- net GND: now also R7.2, RV1.2, RV1.3, U5.5 (0V), U9.11 (5A), J14.2 (Pin_2), J15.2 (Pin_2), R5.1
- net RUN_OK: no longer U9.11 (5A)
- net U1_VDDM: now reaches C10.2, C11.1, U1.6 (VDDM)
- net at R7.1: now also D4.1 (K)
- net GATE_PRE: now reaches Q2.1, R10.1, R9.1
- net PRE_DRAIN: now reaches Q2.2, R1.2
- net BUCK_IN: now reaches C6.1, U5.3 (Vin)
- net BUCK_IN: now also D1.1 (K), D3.1 (K)
- net U2_VDDM: now reaches C12.2, C13.1, U2.6 (VDDM)
- net U2_VDDH: now reaches C12.1, U2.7 (VDDH)
- net BATT_IN: now reaches F1.1, F1.3, J13.P (POS)
- net U1_VDDH: now reaches C10.1, U1.7 (VDDH)
- net EN_BLEED: no longer names the net of U9.10 (5Y)
- net POR_N renamed reset_N
- net POR_RC renamed reset_rc
- no-connect marks 5 -> 6
Other:
- note added: "dishcahrge"
- note removed: "discharge circuit"
- note removed: "masterswitch circut"
- moved on the sheet: C1, C10, C11, C16, C17, C2, C21, C3, C4, D1, D3, Q2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
