File: PDC_new (2)/PDC_new (2).kicad_sch (KiCad schematic)
At the start: 96 parts, among them J1 Conn_01x02_Pin, J10 Conn_01x02_Pin, J12 Conn_01x02_Pin, J13 XT90PW-F, J14 B2B-XH-A__LF__SN_, J15 Conn_01x02, J2 Conn_01x02_Pin, J3 Conn_01x02_Pin, J4 Conn_01x02_Pin, J5 Conn_01x02_Pin, J6 Conn_01x02_Pin, J7 Conn_01x02_Pin, J8 Conn_01x02_Pin, J9 Conn_01x02_Pin, Q1 BSS123, Q2 IRF540NSTRLPBF, U1 TPSI3050QDWZRQ1, U10 LM393LVDR, U11 IPB017N10N5ATMA1, U12 IPB017N10N5ATMA1, U14 IPB017N10N5ATMA1, U2 TPSI3050QDWZRQ1, U3 TPSI3050QDWZRQ1, U4 74HC74, U5 URB4805LD-60WR3, U6 IPB017N10N5ATMA1, U7 TLC555CDR, U8 SN74HC08D, U9 SN74HC14DR

Commit message: Update PDC_new (2) with full PCB layout and latest schematic
Replace the placeholder PDC_new (2) project with the working copy,
including the routed PCB, updated schematic/project settings and the
DRC/ERC report.

Co-Authored-By: Claude Opus 5.5 <noreply@anthropic.com>
Connections:
- net CMP_FILT: now also R25.2; no longer R25.1
- net U1_VDDM: now reaches C10.2, C11.1, U1.6 (VDDM)
- net at C20.2, R26.2, U10.1 (OUT1): now also R25.1; no longer R25.2
- net GATE_PRE: now reaches Q2.1, R10.1, R9.1
- net PRE_DRAIN: now reaches Q2.2, R1.2
- net PRE_FUSE: now reaches F3.2, F3.4, R1.1
- net BUCK_IN: now reaches C6.1, F2.2, F2.4, U5.3 (Vin)
- net BUCK_OR: now reaches D1.1 (K), D3.1 (K), F2.1, F2.3
- net U2_VDDM: now reaches C12.2, C13.1, U2.6 (VDDM)
- net U2_VDDH: now reaches C12.1, U2.7 (VDDH)
- net BATT_IN: now reaches F1.1, F1.3, J13.P (POS)
- net U1_VDDH: now reaches C10.1, U1.7 (VDDH)
Other:
- note added: "Bat+"
- note added: "Bus+"
- note added: "short pin1,2"
- note removed: "bus capacitors"
- note removed: "charging circut"
- note removed: "comparator"
- note removed: "discharge circuit"
- note removed: "mainbus circut"
- note removed: "masterswitch circut"
- moved on the sheet: C1, C10, C11, C12, C13, C14, C15, C16, C17, C18, C19, C2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

Commit message: Replace PDC_new (2) schematic with correct version
Co-Authored-By: Claude Opus 5.5 <noreply@anthropic.com>
Connections:
- net CMP_FILT: now also R25.1; no longer R25.2
- net at C20.2, R26.2, U10.1 (OUT1): now also R25.2; no longer R25.1
- net BATT_IN: no longer names the net of F1.1, F1.3, J13.P (POS)
- net BUCK_IN: no longer names the net of C6.1, F2.2, F2.4, U5.3 (Vin)
- net BUCK_OR: no longer names the net of D1.1 (K), D3.1 (K), F2.1, F2.3
- net GATE_PRE: no longer names the net of Q2.1, R10.1, R9.1
- net PRE_DRAIN: no longer names the net of Q2.2, R1.2
- net PRE_FUSE: no longer names the net of F3.2, F3.4, R1.1
- net U1_VDDH: no longer names the net of C10.1, U1.7 (VDDH)
- net U1_VDDM: no longer names the net of C10.2, C11.1, U1.6 (VDDM)
- net U2_VDDH: no longer names the net of C12.1, U2.7 (VDDH)
- net U2_VDDM: no longer names the net of C12.2, C13.1, U2.6 (VDDM)
Other:
- note added: "bus capacitors"
- note added: "charging circut"
- note added: "comparator"
- note added: "discharge circuit"
- note added: "mainbus circut"
- note added: "masterswitch circut"
- note removed: "Bat+"
- note removed: "Bus+"
- note removed: "short pin1,2"
- moved on the sheet: C1, C10, C11, C12, C13, C14, C15, C16, C17, C18, C19, C2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
