File: PDC_new (2)/PDC_new (2).kicad_sch (KiCad schematic)
At the start: 96 parts, among them J1 Conn_01x02_Pin, J10 Conn_01x02_Pin, J12 Conn_01x02_Pin, J13 XT90PW-F, J14 B2B-XH-A__LF__SN_, J15 Conn_01x02, J2 Conn_01x02_Pin, J3 Conn_01x02_Pin, J4 Conn_01x02_Pin, J5 Conn_01x02_Pin, J6 Conn_01x02_Pin, J7 Conn_01x02_Pin, J8 Conn_01x02_Pin, J9 Conn_01x02_Pin, Q1 BSS123, Q2 IRF540NSTRLPBF, U1 TPSI3050QDWZRQ1, U10 LM393LVDR, U11 IPB017N10N5ATMA1, U12 IPB017N10N5ATMA1, U14 IPB017N10N5ATMA1, U2 TPSI3050QDWZRQ1, U3 TPSI3050QDWZRQ1, U4 74HC74, U5 URB4805LD-60WR3, U6 IPB017N10N5ATMA1, U7 TLC555CDR, U8 SN74HC08D, U9 SN74HC14DR

Commit message: Started routing in PCB editor and fixed the charging connector and MOSFET mistake in schematic
Co-Authored-By: Claude Opus 5.5 <noreply@anthropic.com>
Parts:
- removed J15: Conn_01x02, Connector_JST:JST_XH_B2B-XH-A_1x02_P2.50mm_Vertical, symbol Connector_Generic:Conn_01x02
- added U13: XT90PW(2+2)-M.G.Y, XT90I(2+2)PW-M:CONN-TH_XT90PW2X2-MGY, symbol XT90I(2+2)PW-M:XT90PW(2+2)-M.G.Y
Connections:
- net BATT+: now also U11.7, U12.7, U14.7, U6.7, U13.2; no longer U11.4, U12.4, U14.4, U6.4
- net BUS+: now also U11.4, U12.4, U14.4, U6.4; no longer U11.7, U12.7, U14.7, U6.7
- net DET: now also U13.5
- net GND: now also U13.1, U13.6
- no-connect marks 3 -> 5
Other:
- moved on the sheet: R31
