File: PDC_new (2)/PDC_new (2).kicad_sch (KiCad schematic)
At the start: 96 parts, among them J1 Conn_01x02_Pin, J10 Conn_01x02_Pin, J12 Conn_01x02_Pin, J13 XT90PW-F, J14 B2B-XH-A__LF__SN_, J15 Conn_01x02, J2 Conn_01x02_Pin, J3 Conn_01x02_Pin, J4 Conn_01x02_Pin, J5 Conn_01x02_Pin, J6 Conn_01x02_Pin, J7 Conn_01x02_Pin, J8 Conn_01x02_Pin, J9 Conn_01x02_Pin, Q1 BSS123, Q2 IRF540NSTRLPBF, U1 TPSI3050QDWZRQ1, U10 LM393LVDR, U11 IPB017N10N5ATMA1, U12 IPB017N10N5ATMA1, U14 IPB017N10N5ATMA1, U2 TPSI3050QDWZRQ1, U3 TPSI3050QDWZRQ1, U4 74HC74, U5 URB4805LD-60WR3, U6 IPB017N10N5ATMA1, U7 TLC555CDR, U8 SN74HC08D, U9 SN74HC14DR

Commit message: Route PDC_new (2) PCB and swap JST/switch for XT90PW(2+2) connector
Schematic:
- Replace the two JST XH (B2B-XH-A) connectors and the TS-1187A
  tactile switch with a single XT90PW(2+2)-M.G.Y power+signal connector
- Update related passives, power symbols and net labels

PCB:
- Sync footprints with the schematic (drop JST XH and TS-1187A,
  add CONN-TH_XT90PW2X2-MGY)
- Add first routing pass: ~290 track segments and 6 copper zones

Project:
- Adjust design rules: hole clearance 0.25 mm, min via 0.5 mm /
  0.1 mm annular ring, min text 0.8 mm / 0.08 mm thickness
- Clear predefined track width and diff-pair presets

Co-Authored-By: Claude Opus 5.5 <noreply@anthropic.com>
Parts:
- removed C24: 2.2µF, Capacitor_SMD:C_0805_2012Metric, symbol Device:C
- removed J14: B2B-XH-A__LF__SN_, Connector_JST:JST_XH_B2B-XH-A_1x02_P2.50mm_Vertical, symbol B2B-XH-A__LF__SN_:B2B-XH-A__LF__SN_
- removed J15: Conn_01x02, Connector_JST:JST_XH_B2B-XH-A_1x02_P2.50mm_Vertical, symbol Connector_Generic:Conn_01x02
- removed R28, R29: 10k, Resistor_SMD:R_0805_2012Metric, symbol Device:R
- removed S1: TS-1187A-B-A-B, TS-1187A-B-A-B:SW_TS-1187A-B-A-B, symbol TS-1187A-B-A-B:TS-1187A-B-A-B
- added J11: XT90PW(2+2)-M.G.Y, XT90PW(2+2)-M.G.Y:CONN-TH_XT90PW2X2-MGY, symbol XT90I(2+2)PW-M:XT90PW(2+2)-M.G.Y
Connections:
- net MSTR_FILT is gone; now on net GND: U9.5 (3A)
- net BATT+: now also F3.2, F3.4, U11.7, U12.7, U14.7, U6.7, J11.2; no longer F3.1, F3.3, U11.4, U12.4, U14.4, U6.4
- net BUS+: now also U11.4, U12.4, U14.4, U6.4; no longer U11.7, U12.7, U14.7, U6.7
- net DET: now also J11.5
- net GND: now also RV1.2, RV1.3, U5.5 (0V), J11.1, J11.6
- net U1_VDDM: now reaches C10.2, C11.1, U1.6 (VDDM)
- net GATE_PRE: now reaches Q2.1, R10.1, R9.1
- net PRE_DRAIN: now reaches Q2.2, R1.2
- net BUCK_IN: now reaches C6.1, F2.2, F2.4, U5.3 (Vin)
- net BUCK_OR: now reaches D1.1 (K), D3.1 (K), F2.1, F2.3
- net U2_VDDM: now reaches C12.2, C13.1, U2.6 (VDDM)
- net U2_VDDH: now reaches C12.1, U2.7 (VDDH)
- net BATT_IN: now reaches F1.1, F1.3, J13.P (POS)
- net U1_VDDH: now reaches C10.1, U1.7 (VDDH)
- new net PRE_FUSE: F3.1, F3.3, R1.1
- no-connect marks 3 -> 5
Other:
- note removed: "masterswitch circut"
- moved on the sheet: R31

Commit message: Update PDC_new (2) schematic
Remove C8, C14, C15, D6, F2, F3, Q1, R2, R7, R8, R19, R30, U3; add D4, R5.

Co-Authored-By: Claude Opus 5.5 <noreply@anthropic.com>
Parts:
- removed C14: 470nF, Capacitor_SMD:C_1206_3216Metric, symbol Device:C
- removed C15: 470nF, Capacitor_SMD:C_0805_2012Metric, symbol Device:C
- removed C8: 1µF, Capacitor_SMD:C_0805_2012Metric, symbol Device:C
- removed D6: LED, LED_SMD:LED_0805_2012Metric, symbol Device:LED
- removed F2, F3: 3568-15, Fuse:Fuseholder_Blade_Mini_Keystone_3568, symbol 3568-15:3568-15
- removed Q1: BSS123, Package_TO_SOT_SMD:SOT-23, symbol Transistor_FET:BSS123
- removed R19: 20k, Resistor_SMD:R_0805_2012Metric, symbol Device:R
- removed R2: 1k, Resistor_THT:R_Axial_Power_L25.0mm_W9.0mm_P30.48mm, symbol Device:R
- removed R30: 22k, Resistor_SMD:R_1206_3216Metric, symbol Device:R
- removed R7: 10, Resistor_SMD:R_0805_2012Metric, symbol Device:R
- removed R8: 10k, Resistor_SMD:R_0805_2012Metric, symbol Device:R
- removed U3: TPSI3050QDWZRQ1, ul_TPSI3050QDWZRQ1:DWZ0008A-MFG, symbol TPSI3050_Q1:TPSI3050QDWZRQ1
- added D4: LED, LED_SMD:LED_0805_2012Metric, symbol Device:LED
- added R5: 1k, Resistor_SMD:R_0805_2012Metric, symbol Device:R
- C12: value 2.2µF -> 4.3µF; footprint Capacitor_SMD:C_0805_2012Metric -> Capacitor_SMD:C_1206_3216Metric
- C13: value 2.2 µF -> 4.3 µF
- C5, C6: value C -> 100uF
Connections:
- net PRE_FUSE is gone; now on net BATT+: R1.1
- net BUS+: now also D4.2 (A), R5.2
- net GND: now also D4.1 (K), R5.1
- net POR_N renamed reset_N
- net POR_RC renamed reset_rc
Other:
- note added: "dishcahrge"
- note removed: "discharge circuit"
- moved on the sheet: C10, C11, C16, C17, C21, Q2, R1, R10, R18, R27, R9, U1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

Commit message: Fix isolated EN_BLEED label in PDC_new (2) schematic
Co-Authored-By: Claude Opus 5.5 <noreply@anthropic.com>
Connections:
- net RUN_OK: no longer U9.11 (5A)
- net EN_BLEED: no longer names the net of U9.10 (5Y)
- no-connect marks 5 -> 7
Changed lines of the file:
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@@
 	)
 	(no_connect
+		(at 355.6 142.24)
+	)
+	(no_connect
 		(at 398.78 55.88)
 	)
 	(no_connect
+		(at 320.04 142.24)
+	)
+	(no_connect
 		(at 492.76 36.83)
 	)
@@
 	(wire
 		(pts
-			(xy 355.6 142.24) (xy 358.14 142.24)
-		)
-		(stroke
-			(width 0)
-			(type default)
-		)
-	)
-	(wire
-		(pts
 			(xy 54.61 254) (xy 54.61 251.46)
 		)
@@
 	(wire
 		(pts
-			(xy 320.04 142.24) (xy 317.5 142.24)
-		)
-		(stroke
-			(width 0)
-			(type default)
-		)
-	)
-	(wire
-		(pts
 			(xy 219.71 246.38) (xy 219.71 243.84)
 		)
@@
 		)
 	)
-	(label "RUN_OK"
-		(at 317.5 142.24 180)
-		(effects
-			(font
-				(size 1.27 1.27)
-			)
-			(justify right bottom)
-		)
-	)
 	(label "reset_N"
 		(at 450.85 138.43 180)
@@
 		)
 	)
-	(label "EN_BLEED"
-		(at 358.14 142.24 0)
-		(effects
-			(font
-				(size 1.27 1.27)
-			)
-			(justify left bottom)
-		)
-	)
 	(label "BUS+"
 		(at 377.19 251.46 180)
@@
 		(property "Footprint" "XT90PW-F:AMASS_XT90PW-F"
 			(at 34.29 185.42 0)
-			(hide yes)
 			(show_name no)
 			(do_not_autoplace no)

Commit message: Update PDC_new (2) schematic
Co-Authored-By: Claude Opus 5.5 <noreply@anthropic.com>
Parts:
- added R7: 22k, Resistor_SMD:R_1206_3216Metric_Pad1.30x1.75mm_HandSolder, symbol Device:R
- C10, C11, C9: footprint Capacitor_SMD:C_0805_2012Metric -> LED_SMD:LED_0805_2012Metric_Pad1.15x1.40mm_HandSolder
- C12, C13: footprint Capacitor_SMD:C_1206_3216Metric -> Capacitor_SMD:C_1206_3216Metric_Pad1.33x1.80mm_HandSolder
- C16, C17, C18, C19, C20, C21, C22, C23, C25, C26: footprint Capacitor_SMD:C_0805_2012Metric -> Capacitor_SMD:C_0805_2012Metric_Pad1.18x1.45mm_HandSolder
- R10, R11, R12, R13, R14, R15, R16, R17, R18, R20, R21, R22, R23, R24, R25, R26, R27, R31, R4, R5, R6, R9: footprint Resistor_SMD:R_0805_2012Metric -> Resistor_SMD:R_0805_2012Metric_Pad1.20x1.40mm_HandSolder
- R3: footprint Resistor_SMD:R_0805_2012Metric -> Resistor_SMD:R_1206_3216Metric_Pad1.30x1.75mm_HandSolder
Connections:
- net BUCK_OR is gone; now on net BUCK_IN: D1.1 (K), D3.1 (K)
- net GND: now also U9.11 (5A), R7.2; no longer D4.1 (K)
- new net: D4.1 (K), R7.1
- no-connect marks 7 -> 6
Other:
- moved on the sheet: D1, D3, R10

Commit message: Change R5 to axial power THT footprint and update PCB layout
- Schematic: R5 (1k) footprint changed from R_0805 SMD hand-solder to
  Resistor_THT:R_Axial_Power_L25.0mm_W9.0mm_P30.48mm.
- PCB: board re-synced with updated footprints, re-routed tracks, added
  vias and copper zones.
- Project: default pad size updated to 1.95 x 0.6 mm SMD.

Co-Authored-By: Claude Opus 5.5 <noreply@anthropic.com>
Parts:
- R5: footprint Resistor_SMD:R_0805_2012Metric_Pad1.20x1.40mm_HandSolder -> Resistor_THT:R_Axial_Power_L25.0mm_W9.0mm_P30.48mm
Changed lines of the file:
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@@
 			)
 		)
-		(property "Footprint" "Resistor_SMD:R_0805_2012Metric_Pad1.20x1.40mm_HandSolder"
+		(property "Footprint" "Resistor_THT:R_Axial_Power_L25.0mm_W9.0mm_P30.48mm"
 			(at 97.028 303.53 90)
 			(hide yes)

Commit message: Update PDC_new (2) schematic
Co-Authored-By: Claude Opus 5.5 <noreply@anthropic.com>
Parts:
- added J14, J15: Conn_01x02_Pin, Connector_AMASS:AMASS_XT60PW-F_1x02_P7.20mm_Horizontal, symbol Connector:Conn_01x02_Pin
- J13: value XT90PW-F -> QS8; footprint XT90PW-F:AMASS_XT90PW-F -> QS8_S_Connectors:QS8-S-M_Vertical_DirectCup
- R5: value 1k -> 10k
Connections:
- net BUS+: now also J14.1 (Pin_1), J15.1 (Pin_1)
- net GND: now also J14.2 (Pin_2), J15.2 (Pin_2)
Other:
- moved on the sheet: C1, C2, C3, C4

Commit message: Update PDC_new (2) schematic, PCB layout and project settings
Co-Authored-By: Claude Opus 5.5 <noreply@anthropic.com>
Parts:
- removed J13: QS8, QS8_S_Connectors:QS8-S-M_Vertical_DirectCup, symbol XT90I:XT90PW-F
- added J13: Conn_01x02_Pin, QS8_S_Connectors:QS8-S-M_Vertical_DirectCup, symbol Connector:Conn_01x02_Pin
Connections:
- net BATT_IN: now also J13.1 (Pin_1)
- net GND: now also J13.2 (Pin_2)
Other:
- moved on the sheet: F1
