File: PDC_new (2)/PDC_new (2).kicad_pcb (KiCad board)
At the start: 2 copper layers, 96 parts, among them J1 Conn_01x02_Pin, J10 Conn_01x02_Pin, J12 Conn_01x02_Pin, J13 XT90PW-F, J14 B2B-XH-A__LF__SN_, J15 Conn_01x02, J2 Conn_01x02_Pin, J3 Conn_01x02_Pin, J4 Conn_01x02_Pin, J5 Conn_01x02_Pin, J6 Conn_01x02_Pin, J7 Conn_01x02_Pin, J8 Conn_01x02_Pin, J9 Conn_01x02_Pin, Q1 BSS123, Q2 IRF540NSTRLPBF, U1 TPSI3050QDWZRQ1, U10 LM393LVDR, U11 IPB017N10N5ATMA1, U12 IPB017N10N5ATMA1, U14 IPB017N10N5ATMA1, U2 TPSI3050QDWZRQ1, U3 TPSI3050QDWZRQ1, U4 74HC74, U5 URB4805LD-60WR3, U6 IPB017N10N5ATMA1, U7 TLC555CDR, U8 SN74HC08D, U9 SN74HC14DR

Commit message: Started routing in PCB editor and fixed the charging connector and MOSFET mistake in schematic
Co-Authored-By: Claude Opus 5.5 <noreply@anthropic.com>
Parts:
- added U13: XT90PW(2+2)-M.G.Y, XT90I(2+2)PW-M:CONN-TH_XT90PW2X2-MGY, F.Cu at (391.0, 331.6)
- moved D7 315.9 mm to (397.5, 307.5)
- moved U5 307.0 mm to (331.5, 325.5)
- moved J6 294.8 mm to (398.2, 173.4), turned to -90 degrees
- moved J7 285.3 mm to (398.2, 190.9), turned to -90 degrees
- moved R31 279.5 mm to (382.1, 305.0)
- moved J8 277.6 mm to (398.2, 208.5), turned to -90 degrees
- moved J9 272.0 mm to (398.2, 226.1), turned to -90 degrees
- moved J12 270.4 mm to (299.0, 325.4), turned to 180 degrees
- moved J10 268.6 mm to (398.2, 243.6), turned to -90 degrees
- moved D1 243.0 mm to (304.4, 293.7)
- moved D3 243.0 mm to (304.4, 298.2)
- moved F2 236.2 mm to (330.5, 282.6)
- moved F4 236.2 mm to (330.5, 299.2)
- moved D2 231.3 mm to (151.4, 325.0)
- moved RV1 231.3 mm to (362.5, 315.0), turned to 90 degrees
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Connections:
- net /BATT_IN renamed Net-(J13-POS)
- net /BUCK_IN renamed Net-(U5-Vin)
- net /BUCK_OR renamed Net-(D1-K)
- net /GATE_PRE renamed Net-(Q2-Pad1)
- net /PRE_DRAIN renamed Net-(Q2-Pad2)
- net /PRE_FUSE renamed Net-(F3-Pad2)
- net /U1_VDDH renamed Net-(U1-VDDH)
- net /U1_VDDM renamed Net-(U1-VDDM)
- net /U2_VDDH renamed Net-(U2-VDDH)
- net /U2_VDDM renamed Net-(U2-VDDM)
- J15 pad 1: /DET -> /BATT+
- R25 pad 1: Net-(U10A-OUT1) -> /CMP_FILT
- R25 pad 2: /CMP_FILT -> Net-(U10A-OUT1)
- U11 pad 4: /BATT+ -> /BUS+
- U11 pad 7: /BUS+ -> /BATT+
- U12 pad 4: /BATT+ -> /BUS+
- U12 pad 7: /BUS+ -> /BATT+
- U14 pad 4: /BATT+ -> /BUS+
- U14 pad 7: /BUS+ -> /BATT+
- U6 pad 4: /BATT+ -> /BUS+
- U6 pad 7: /BUS+ -> /BATT+

Commit message: pcb: continue routing, add board outline, remove stray J15
Remove J15 footprint, which has no matching symbol in the schematic.
Mirror the same board into the top-level PDC_new.kicad_pcb.

Co-Authored-By: Claude Opus 5.5 <noreply@anthropic.com>
Parts:
- removed J15: Conn_01x02, Connector_JST:JST_XH_B2B-XH-A_1x02_P2.50mm_Vertical
- moved C6 196.5 mm to (341.1, 308.0)
- moved F1 189.6 mm to (243.0, 280.8)
- moved F3 184.7 mm to (281.5, 251.3)
- moved R4 178.8 mm to (308.9, 254.5)
- moved R6 176.4 mm to (304.0, 260.5)
- moved C18 170.2 mm to (345.0, 248.0)
- moved D5 162.2 mm to (314.0, 243.5), turned to 90 degrees
- moved C22 161.2 mm to (347.0, 231.5)
- moved R24 159.1 mm to (319.0, 236.4), turned to 90 degrees
- moved R22 158.0 mm to (308.9, 260.5)
- moved C25 154.9 mm to (330.0, 248.0)
- moved C19 146.8 mm to (319.0, 243.0), turned to 90 degrees
- moved R21 146.7 mm to (303.9, 255.0)
- moved C26 142.0 mm to (331.5, 232.0)
- moved C23 139.4 mm to (334.5, 216.0)
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Routing:
- net Net-(U3-VDDH): track 0.00 -> 3.13 mm
